File: uStar/uStar_v1.brd (EAGLE design)
At the start: 85 x 40 mm, 30 parts, among them IC1 INA138, X1 BU-SMA-V

Commit message: added changes submitted by Ben
Parts:
- added U$6: OPENLOG, LearningByMaking:OPENLOG
- PAD1, PAD2, PAD3, PAD4: value (none) -> (none)
- moved X1 0.80 mm to (4.57, 29.0)
Connections:
- net +3V3: now also GPS.2, GPS.5, U$3.VIN, U$4.VCC, U$5.P$4
- net VCC: no longer GPS.2, GPS.5, U$3.VIN, U$4.VCC, U$5.P$4
- net VREAD: now also U$1.P21
Routing:
- net GND: track 185.7 -> 0.00 mm, vias 1 -> 0
- net +3V3: track 20.5 -> 158.8 mm, vias 0 -> 7
- net VCC: track 185.1 -> 131.0 mm, vias 10 -> 6
- net VREAD: track 12.4 -> 25.4 mm
- net N$7: track 43.8 -> 32.1 mm, vias 2 -> 1
- net GPS_TX: track 39.2 -> 31.3 mm, vias 4 -> 2
- net 1WIRE: track 141.1 -> 144.1 mm
- net CLK: track 49.5 -> 50.9 mm
- net N$1: track 34.8 -> 33.6 mm
- net N$2: track 33.2 -> 32.1 mm
- net 9DOF_SDA: track 18.2 -> 17.1 mm
- net N$4: track 11.0 -> 12.0 mm
- net N$5: track 11.2 -> 12.2 mm
- net 9DOF_SCL: track 15.5 -> 14.6 mm
- net GPS_RX: track 21.2 -> 21.7 mm
