File: uStar/uStar_v1.sch (EAGLE design)
At the start: 30 parts, among them IC1 INA138, X1 BU-SMA-V

Commit message: added changes submitted by Ben
Parts:
- added U$6: OPENLOG, LearningByMaking:OPENLOG
- PAD1, PAD2, PAD3, PAD4: value (none) -> (none)
Connections:
- net +3V3: now also GPS-2.S, GPS-5.S, U$3.VIN, U$4.VIN, U$5.VCC
- net VCC: no longer GPS-2.S, GPS-5.S, U$3.VIN, U$4.VIN, U$5.VCC
- net VREAD: now also U$1.ADC7
Changed lines of the file:
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@@
 <part name="U$4" library="LearningByMaking" deviceset="TMP_EXT" device=""/>
 <part name="GPS" library="con-jst2" deviceset="SM06B-SSR-H-TB" device=""/>
-<part name="PAD1" library="wirepad" deviceset="1,6/0,9" device=""/>
-<part name="PAD2" library="wirepad" deviceset="1,6/0,9" device=""/>
-<part name="PAD3" library="wirepad" deviceset="1,6/0,9" device=""/>
-<part name="PAD4" library="wirepad" deviceset="1,6/0,9" device=""/>
+<part name="PAD1" library="wirepad" deviceset="1,6/0,9" device="" value=" "/>
+<part name="PAD2" library="wirepad" deviceset="1,6/0,9" device="" value=" "/>
+<part name="PAD3" library="wirepad" deviceset="1,6/0,9" device="" value=" "/>
+<part name="PAD4" library="wirepad" deviceset="1,6/0,9" device="" value=" "/>
+<part name="U$6" library="LearningByMaking" deviceset="OPENLOG" device=""/>
 </parts>
 <sheets>
@@
 <instance part="PAD3" gate="1" x="45.72" y="152.4"/>
 <instance part="PAD4" gate="1" x="45.72" y="157.48"/>
+<instance part="U$6" gate="G$1" x="68.58" y="22.86"/>
 </instances>
 <busses>
@@
 <pinref part="+3V2" gate="G$1" pin="+3V3"/>
 </segment>
+<segment>
+<wire x1="27.94" y1="101.6" x2="33.02" y2="101.6" width="0.1524" layer="91"/>
+<label x="33.02" y="101.6" size="1.27" layer="95" xref="yes"/>
+<pinref part="U$4" gate="G$1" pin="VIN"/>
+</segment>
+<segment>
+<wire x1="48.26" y1="73.66" x2="48.26" y2="76.2" width="0.1524" layer="91"/>
+<pinref part="U$5" gate="G$1" pin="VCC"/>
+<wire x1="48.26" y1="76.2" x2="53.34" y2="76.2" width="0.1524" layer="91"/>
+<label x="48.26" y="73.66" size="1.27" layer="95" rot="R270" xref="yes"/>
+</segment>
+<segment>
+<wire x1="88.9" y1="58.42" x2="93.98" y2="58.42" width="0.1524" layer="91"/>
+<wire x1="93.98" y1="58.42" x2="93.98" y2="53.34" width="0.1524" layer="91"/>
+<wire x1="93.98" y1="53.34" x2="109.22" y2="53.34" width="0.1524" layer="91"/>
+<wire x1="109.22" y1="60.96" x2="93.98" y2="60.96" width="0.1524" layer="91"/>
+<wire x1="93.98" y1="60.96" x2="93.98" y2="58.42" width="0.1524" layer="91"/>
+<junction x="93.98" y="58.42"/>
+<label x="88.9" y="58.42" size="1.27" layer="95" rot="R180" xref="yes"/>
+<pinref part="GPS" gate="-2" pin="S"/>
+<pinref part="GPS" gate="-5" pin="S"/>
+</segment>
+<segment>
+<pinref part="U$3" gate="G$1" pin="VIN"/>
+<wire x1="7.62" y1="170.18" x2="12.7" y2="170.18" width="0.1524" layer="91"/>
+<label x="7.62" y="170.18" size="1.27" layer="95" rot="R180" xref="yes"/>
+</segment>
 </net>
 <net name="1WIRE" class="0">
@@
 <pinref part="P+1" gate="VCC" pin="VCC"/>
 </segment>
-<segment>
-<pinref part="U$3" gate="G$1" pin="VIN"/>
-<wire x1="7.62" y1="170.18" x2="12.7" y2="170.18" width="0.1524" layer="91"/>
-<label x="7.62" y="170.18" size="1.27" layer="95" rot="R180" xref="yes"/>
-</segment>
-<segment>
-<wire x1="27.94" y1="101.6" x2="33.02" y2="101.6" width="0.1524" layer="91"/>
-<label x="33.02" y="101.6" size="1.27" layer="95" xref="yes"/>
-<pinref part="U$4" gate="G$1" pin="VIN"/>
-</segment>
-<segment>
-<wire x1="48.26" y1="73.66" x2="48.26" y2="76.2" width="0.1524" layer="91"/>
-<pinref part="U$5" gate="G$1" pin="VCC"/>
-<wire x1="48.26" y1="76.2" x2="53.34" y2="76.2" width="0.1524" layer="91"/>
-<label x="48.26" y="73.66" size="1.27" layer="95" rot="R270" xref="yes"/>
-</segment>
-<segment>
-<wire x1="88.9" y1="58.42" x2="93.98" y2="58.42" width="0.1524" layer="91"/>
-<wire x1="93.98" y1="58.42" x2="93.98" y2="53.34" width="0.1524" layer="91"/>
-<wire x1="93.98" y1="53.34" x2="109.22" y2="53.34" width="0.1524" layer="91"/>
-<wire x1="109.22" y1="60.96" x2="93.98" y2="60.96" width="0.1524" layer="91"/>
-<wire x1="93.98" y1="60.96" x2="93.98" y2="58.42" width="0.1524" layer="91"/>
-<junction x="93.98" y="58.42"/>
-<label x="88.9" y="58.42" size="1.27" layer="95" rot="R180" xref="yes"/>
-<pinref part="GPS" gate="-2" pin="S"/>
-<pinref part="GPS" gate="-5" pin="S"/>
-</segment>
 </net>
 <net name="VREAD" class="0">
@@
 <label x="162.56" y="88.9" size="1.778" layer="95" xref="yes"/>
 <junction x="160.02" y="88.9"/>
+</segment>
+<segment>
+<wire x1="127" y1="165.1" x2="129.54" y2="165.1" width="0.1524" layer="91"/>
+<label x="127" y="165.1" size="1.778" layer="95" rot="R180" xref="yes"/>
+<pinref part="U$1" gate="G$1" pin="ADC7"/>
 </segment>
 </net>
@@
 </sheet>
 </sheets>
+<errors>
+</errors>
 </schematic>
 </drawing>
